File: board_sierra.sch (KiCad schematic (older format))
At the start: 244 parts, among them M1 S25FL256L, M2 S25FL256L, M3 S25FL256L, M4 CY15B102Q, M5 CY15B102Q, M6 CY15B102Q, Q1 TPS22965-Q1, Q2 TPS22965-Q1, Q3 TPS22965-Q1, U1 STM32L496ZGTx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

Commit message: sync with library
Parts:
- D4: footprint VST104_footprints:D_SMD_SOD523_1.2x0.8mm -> VST104_footprints:D_SOD-523_1.2x0.8mm
- H1, H2: footprint VST104_footprints:ESQ-129-39-x-D -> VST104_footprints:ESQ-126-39-x-D
Changed lines of the file:
@@
 F 0 "H2" H 21000 14200 50  0000 C CNN
 F 1 "Conn_02x26_Odd_Even" H 21000 11500 50  0001 C CNN
-F 2 "VST104_footprints:ESQ-129-39-x-D" H 20950 12900 50  0001 C CNN
-F 3 "~" H 20950 12900 50  0001 C CNN
+F 2 "VST104_footprints:ESQ-126-39-x-D" H 20950 12900 50  0001 C CNN
+F 3 "https://www.mouser.sk/datasheet/2/527/esq_th-1369982.pdf" H 20950 12900 50  0001 C CNN
 	1    20950 12900
 	1    0    0    -1
@@
 F 0 "H1" H 21000 11250 50  0000 C CNN
 F 1 "Conn_02x26_Odd_Even" H 21000 8550 50  0001 C CNN
-F 2 "VST104_footprints:ESQ-129-39-x-D" H 20950 9950 50  0001 C CNN
-F 3 "~" H 20950 9950 50  0001 C CNN
+F 2 "VST104_footprints:ESQ-126-39-x-D" H 20950 9950 50  0001 C CNN
+F 3 "https://www.mouser.sk/datasheet/2/527/esq_th-1369982.pdf" H 20950 9950 50  0001 C CNN
 	1    20950 9950
 	1    0    0    -1
@@
 F 0 "D4" V 21550 2400 50  0000 L CNN
 F 1 "BZT52C3V3TQ-7-F" H 21050 2750 50  0000 L CNN
-F 2 "VST104_footprints:D_SMD_SOD523_1.2x0.8mm" H 21550 2600 50  0001 C CNN
+F 2 "VST104_footprints:D_SOD-523_1.2x0.8mm" H 21550 2600 50  0001 C CNN
 F 3 "https://www.mouser.sk/datasheet/2/115/ds30502-1142513.pdf" H 21550 2600 50  0001 C CNN
 	1    21550 2600

Commit message: L1 to 0603
Parts:
- L1: footprint VST104_footprints:L_SMD_0402 -> VST104_footprints:L_SMD_0603
Changed lines of the file:
@@
 F 0 "L1" V 3800 1300 50  0000 C CNN
 F 1 "10u" V 4000 1300 50  0000 C CNN
-F 2 "VST104_footprints:L_SMD_0402" H 3900 1300 50  0001 C CNN
+F 2 "VST104_footprints:L_SMD_0603" H 3900 1300 50  0001 C CNN
 F 3 "https://www.mouser.sk/datasheet/2/281/JELF243A-0169-1324396.pdf" H 3900 1300 50  0001 C CNN
 	1    3900 1300

Commit message: power management update
Parts:
- removed D4: BZT52C3V3TQ-7-F, VST104_footprints:D_SOD-523_1.2x0.8mm, symbol Device:D_Zener
- removed R75: 47k, VST104_footprints:R_SMD_0402, symbol Device:R
- removed R81: 330, VST104_footprints:R_SMD_0402, symbol Device:R
- C56, C57: symbol Device:CP -> Device:C
- D1, D2, D3: value CDBQR40 -> CDBQR40-HF
- EF1, EF2: symbol VST104:TPS25940-Q1 -> VST104:TPS25940x
- LG1: symbol VST104:74LVC1G11-Q100 -> VST104:74LVC1G11
- Q1: symbol VST104:TPS22965-Q1 -> board_sierra-rescue:TPS22965-Q1-VST104
- Q2, Q3: value TPS22965-Q1 -> TPS22965W-Q1; symbol VST104:TPS22965-Q1 -> VST104:TPS22965x
- R53: value 100k -> 10k
- R76: value 56k -> 10k
Connections:
- net at LG1.4 (Y): now also Q2.3 (EN), Q3.3 (EN), R76.1
Other:
- moved on the sheet: C39, C40, C49, C50, C51, C52, C55, C60, C61, C66, C67, C70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
