File: board_sierra.sch (KiCad schematic (older format))
At the start: 241 parts, among them M1 S25FL256L, M2 S25FL256L, M3 S25FL256L, M4 CY15B102Q, M5 CY15B102Q, M6 CY15B102Q, Q1 TPS22965-Q1, Q2 TPS22965W-Q1, Q3 TPS22965W-Q1, U1 STM32L496ZGTx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

Commit message: libraries updated
Parts:
- Q1: symbol board_sierra-rescue:TPS22965-Q1-VST104 -> VST104:TPS22965x
Changed lines of the file:
@@
 TEMP_VDD
 $Comp
-L board_sierra-rescue:TPS22965-Q1-VST104 Q1
+L VST104:TPS22965x Q1
 U 1 1 61860A10
 P 9600 1900
-F 0 "Q1" H 9850 2300 50  0000 C CNN
+F 0 "Q1" H 9850 2450 50  0000 C CNN
 F 1 "TPS22965-Q1" H 9850 1850 50  0000 C CNN
 F 2 "VST104_footprints:WSON-8_2.0x2.0mm_EPV" H 9850 2350 50  0001 C CNN

Commit message: MCU resin hole added
Parts:
- added RH1: ResinHole, VST104_footprints:MountingHole_1.2mm, symbol Mechanical:MountingHole
Other:
- moved on the sheet: MH2, MH4, TP17, TP18
Changed lines of the file:
@@
 Sheet 1 1
 Title "VST104 single OBCboard"
-Date "2020-09-14"
+Date "2021-03-03"
 Rev "1.1"
 Comp "Vision Space Technologies"
@@
 U 1 1 5E50DEC4
 P 19150 15000
-F 0 "MH3" H 19250 15003 50  0000 L CNN
+F 0 "MH3" H 19250 15050 50  0000 L CNN
 F 1 "MountingHole_Pad" H 19250 14958 50  0001 L CNN
 F 2 "VST104_footprints:MountingHole_3.2mm_M3_Pad_Via" H 19150 15000 50  0001 C CNN
@@
 $EndComp
 NoConn ~ 18800 15100
-NoConn ~ 19350 15300
-NoConn ~ 18950 15300
+NoConn ~ 19350 15250
+NoConn ~ 18950 15250
 $Comp
 L Mechanical:MountingHole_Pad MH4
 U 1 1 5E50E2B0
-P 19350 15200
-F 0 "MH4" H 19450 15203 50  0000 L CNN
-F 1 "MountingHole_Pad" H 19450 15158 50  0001 L CNN
-F 2 "VST104_footprints:MountingHole_3.2mm_M3_Pad_Via" H 19350 15200 50  0001 C CNN
-F 3 "~" H 19350 15200 50  0001 C CNN
-	1    19350 15200
+P 19350 15150
+F 0 "MH4" H 19400 15100 50  0000 L CNN
+F 1 "MountingHole_Pad" H 19450 15108 50  0001 L CNN
+F 2 "VST104_footprints:MountingHole_3.2mm_M3_Pad_Via" H 19350 15150 50  0001 C CNN
+F 3 "~" H 19350 15150 50  0001 C CNN
+	1    19350 15150
 	1    0    0    -1
 $EndComp
@@
 L Mechanical:MountingHole_Pad MH2
 U 1 1 5E50E4A0
-P 18950 15200
-F 0 "MH2" H 19050 15203 50  0000 L CNN
-F 1 "MountingHole_Pad" H 19050 15158 50  0001 L CNN
-F 2 "VST104_footprints:MountingHole_3.2mm_M3_Pad_Via" H 18950 15200 50  0001 C CNN
-F 3 "~" H 18950 15200 50  0001 C CNN
-	1    18950 15200
+P 18950 15150
+F 0 "MH2" H 19000 15100 50  0000 L CNN
+F 1 "MountingHole_Pad" H 19050 15108 50  0001 L CNN
+F 2 "VST104_footprints:MountingHole_3.2mm_M3_Pad_Via" H 18950 15150 50  0001 C CNN
+F 3 "~" H 18950 15150 50  0001 C CNN
+	1    18950 15150
 	1    0    0    -1
 $EndComp
@@
 U 1 1 5E50E62D
 P 18800 15000
-F 0 "MH1" H 18900 15003 50  0000 L CNN
+F 0 "MH1" H 18900 15050 50  0000 L CNN
 F 1 "MountingHole_Pad" H 18900 14958 50  0001 L CNN
 F 2 "VST104_footprints:MountingHole_3.2mm_M3_Pad_Via" H 18800 15000 50  0001 C CNN
@@
 L power:PWR_FLAG #FLG01
 U 1 1 769BCE2E
-P 20500 15100
-F 0 "#FLG01" H 20500 15175 50  0001 C CNN
-F 1 "PWR_FLAG" H 20500 15273 50  0000 C CNN
-F 2 "" H 20500 15100 50  0001 C CNN
-F 3 "~" H 20500 15100 50  0001 C CNN
-	1    20500 15100
+P 20700 15100
+F 0 "#FLG01" H 20700 15175 50  0001 C CNN
+F 1 "PWR_FLAG" H 20700 15273 50  0000 C CNN
+F 2 "" H 20700 15100 50  0001 C CNN
+F 3 "~" H 20700 15100 50  0001 C CNN
+	1    20700 15100
 	1    0    0    -1
 $EndComp
@@
 L power:PWR_FLAG #FLG02
 U 1 1 76BE42BF
-P 21000 15100
-F 0 "#FLG02" H 21000 15175 50  0001 C CNN
-F 1 "PWR_FLAG" H 21000 15273 50  0000 C CNN
-F 2 "" H 21000 15100 50  0001 C CNN
-F 3 "~" H 21000 15100 50  0001 C CNN
-	1    21000 15100
+P 21200 15100
+F 0 "#FLG02" H 21200 15175 50  0001 C CNN
+F 1 "PWR_FLAG" H 21200 15273 50  0000 C CNN
+F 2 "" H 21200 15100 50  0001 C CNN
+F 3 "~" H 21200 15100 50  0001 C CNN
+	1    21200 15100
 	1    0    0    -1
 $EndComp
@@
 L power:GND #PWR0160
 U 1 1 7700DCCC
-P 21450 15150
-F 0 "#PWR0160" H 21450 14900 50  0001 C CNN
-F 1 "GND" H 21455 14977 50  0000 C CNN
-F 2 "" H 21450 15150 50  0001 C CNN
-F 3 "" H 21450 15150 50  0001 C CNN
-	1    21450 15150
+P 21650 15150
+F 0 "#PWR0160" H 21650 14900 50  0001 C CNN
+F 1 "GND" H 21655 14977 50  0000 C CNN
+F 2 "" H 21650 15150 50  0001 C CNN
+F 3 "" H 21650 15150 50  0001 C CNN
+	1    21650 15150
 	1    0    0    -1
 $EndComp
 Wire Wire Line
-	21450 15100 21450 15150
-Text GLabel 20450 15250 0    50   Input ~ 0
+	21650 15100 21650 15150
+Text GLabel 20650 15250 0    50   Input ~ 0
 SUP_5V
-Text GLabel 20950 15250 0    50   Input ~ 0
+Text GLabel 21150 15250 0    50   Input ~ 0
 SUP_3V3
 Wire Wire Line
-	21000 15250 20950 15250
+	21200 15250 21150 15250
 Wire Wire Line
-	21000 15100 21000 15250
+	21200 15100 21200 15250
 Wire Wire Line
-	20500 15250 20450 15250
+	20700 15250 20650 15250
 Wire Wire Line
-	20500 15100 20500 15250
+	20700 15100 20700 15250
 Wire Notes Line width 10
 	20000 8500 22000 8500
@@
 L power:PWR_FLAG #FLG03
 U 1 1 82F35DD9
-P 21450 15100
-F 0 "#FLG03" H 21450 15175 50  0001 C CNN
-F 1 "PWR_FLAG" H 21450 15273 50  0000 C CNN
-F 2 "" H 21450 15100 50  0001 C CNN
-F 3 "~" H 21450 15100 50  0001 C CNN
-	1    21450 15100
+P 21650 15100
+F 0 "#FLG03" H 21650 15175 50  0001 C CNN
+F 1 "PWR_FLAG" H 21650 15273 50  0000 C CNN
+F 2 "" H 21650 15100 50  0001 C CNN
+F 3 "~" H 21650 15100 50  0001 C CNN
+	1    21650 15100
 	1    0    0    -1
 $EndComp
@@
 L Connector:TestPoint TP17
 U 1 1 6159B948
-P 19650 15050
-F 0 "TP17" H 19708 15168 50  0000 L CNN
-F 1 "GND" H 19708 15077 50  0001 L CNN
-F 2 "VST104_footprints:scope_GND" H 19850 15050 50  0001 C CNN
-F 3 "~" H 19850 15050 50  0001 C CNN
-	1    19650 15050
-	1    0    0    -1
-$EndComp
-$Comp
-L Connector:TestPoint TP18
-U 1 1 6159E270
 P 19950 15050
-F 0 "TP18" H 20008 15168 50  0000 L CNN
+F 0 "TP17" H 20000 15200 50  0000 L CNN
 F 1 "GND" H 20008 15077 50  0001 L CNN
 F 2 "VST104_footprints:scope_GND" H 20150 15050 50  0001 C CNN
@@
 	1    0    0    -1
 $EndComp
+$Comp
+L Connector:TestPoint TP18
+U 1 1 6159E270
+P 20250 15050
+F 0 "TP18" H 20000 15100 50  0000 L CNN
+F 1 "GND" H 20308 15077 50  0001 L CNN
+F 2 "VST104_footprints:scope_GND" H 20450 15050 50  0001 C CNN
+F 3 "~" H 20450 15050 50  0001 C CNN
+	1    20250 15050
+	1    0    0    -1
+$EndComp
 Wire Wire Line
-	19650 15050 19650 15100
+	19950 15050 19950 15100
 Wire Wire Line
-	19650 15100 19800 15100
+	19950 15100 20100 15100
 Wire Wire Line
-	19950 15100 19950 15050
+	20250 15100 20250 15050
 Wire Wire Line
-	19800 15150 19800 15100
-Connection ~ 19800 15100
+	20100 15150 20100 15100
+Connection ~ 20100 15100
 Wire Wire Line
-	19800 15100 19950 15100
+	20100 15100 20250 15100
 $Comp
 L power:GND #PWR0145
 U 1 1 61D45EFF
-P 19800 15150
-F 0 "#PWR0145" H 19800 14900 50  0001 C CNN
-F 1 "GND" H 19805 14977 50  0000 C CNN
-F 2 "" H 19800 15150 50  0001 C CNN
-F 3 "" H 19800 15150 50  0001 C CNN
-	1    19800 15150
+P 20100 15150
+F 0 "#PWR0145" H 20100 14900 50  0001 C CNN
+F 1 "GND" H 20105 14977 50  0000 C CNN
+F 2 "" H 20100 15150 50  0001 C CNN
+F 3 "" H 20100 15150 50  0001 C CNN
+	1    20100 15150
 	1    0    0    -1
 $EndComp
@@
 Wire Wire Line
 	13750 10000 14100 10000
+$Comp
+L Mechanical:MountingHole RH1
+U 1 1 6134FA2A
+P 19600 14950
+F 0 "RH1" H 19700 14950 50  0000 L CNN
+F 1 "ResinHole" H 19700 14905 50  0001 L CNN
+F 2 "VST104_footprints:MountingHole_1.2mm" H 19600 14950 50  0001 C CNN
+F 3 "~" H 19600 14950 50  0001 C CNN
+	1    19600 14950
+	1    0    0    -1
+$EndComp
 Wire Bus Line
 	14200 5400 14200 6450

Commit message: schem. cosmetic updates
Parts:
- C10, C11, C12, C13, C14, C5, C6, C7, C8, C9: symbol Device:C -> Device:C_Small
- D1, D2, D3: value CDBQR40-HF -> Schottky diode
- FB1, FB2: value 120 @ 100M -> 120@100M
- R5: value 22 -> 10k
Connections:
- net labels removed: BOOT
- wire segments 1233 -> 1221
Other:
- note added: "3V3"
- note added: "Microcontroller"
- note added: "reserved I2C1"
- note removed: "- 3V3 tol."
- moved on the sheet: C1, C10, C11, C12, C13, C14, C15, C16, C17, C18, C19, C2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
