File: board_sierra.kicad_pcb (KiCad board)
At the start: 6 copper layers, 90.2 x 95.9 mm, 247 parts, among them M1 S25FL256L, M2 S25FL256L, M3 S25FL256L, M4 CY15B102Q, M5 CY15B102Q, M6 CY15B102Q, Q1 TPS22965-Q1, Q2 TPS22965-Q1, Q3 TPS22965-Q1, U1 STM32L496ZGTx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

Commit message: power management update
Parts:
- removed D4: BZT52C3V3TQ-7-F, VST104_footprints:D_SOD-523_1.2x0.8mm
- removed R75: 47k, VST104_footprints:R_SMD_0402
- removed R81: 330, VST104_footprints:R_SMD_0402
- D1, D2, D3: value CDBQR40 -> CDBQR40-HF
- Q2, Q3: value TPS22965-Q1 -> TPS22965W-Q1
- R53: value 100k -> 10k
- R76: value 56k -> 10k
- moved R76 1.42 mm to (58.2, 57.9), turned to 270 degrees
Connections:
- Q2 pad 3: Net-(Q2-Pad3) -> Net-(LG1-Pad4)
- Q3 pad 3: Net-(Q2-Pad3) -> Net-(LG1-Pad4)
- R76 pad 1: Net-(Q2-Pad3) -> Net-(LG1-Pad4)
Routing:
- net Net-(Q2-Pad3): track 36.0 -> 0.00 mm, vias 4 -> 0
- net Net-(LG1-Pad4): track 1.27 -> 33.4 mm, vias 0 -> 4
- net Net-(D4-Pad1): track 1.28 -> 0.00 mm
- net /I2C2_SDA: track 125.8 -> 124.6 mm
- net /EF1_en: track 11.1 -> 10.1 mm
- net +3V3: track 80.9 -> 80.2 mm
- net +5V: track 168.4 -> 167.8 mm

Commit message: MCU resin hole added
Parts:
- added RH1: ResinHole, VST104_footprints:MountingHole_1.2mm, F.Cu at (42.6, 61.1)
Routing:
- net +5V: track 167.8 -> 168.4 mm
