File: board_sierra.kicad_pcb (KiCad board)
At the start: 6 copper layers, 90.2 x 95.9 mm, 245 parts, among them M1 S25FL256L, M2 S25FL256L, M3 S25FL256L, M4 CY15B102Q, M5 CY15B102Q, M6 CY15B102Q, Q1 TPS22965-Q1, Q2 TPS22965W-Q1, Q3 TPS22965W-Q1, U1 STM32L496ZGTx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

Commit message: schem. cosmetic updates
Parts:
- D1, D2, D3: value CDBQR40-HF -> Schottky diode
- FB1, FB2: value 120 @ 100M -> 120@100M
- R5: value 22 -> 10k
Connections:
- net /BOOT renamed Net-(R5-Pad1)
- net NRST renamed /NRST
- net SW_CLK renamed /SW_CLK
- net SW_DIO renamed /SW_DIO
- net SW_O renamed /SW_O
- net UART5_RX renamed /UART5_RX
- net UART5_TX renamed /UART5_TX
